Commit message: New code structure for v1.0. Added robot specific modules to easily add new robots.

File: assistive_gym/envs/assets/bed_bathing/wiper.urdf (robot description, URDF)
Before this commit: robot wiper, 3 links, 2 joints
Links:
- link cloth: mass 1 -> 0.1
- link handle: mass 1 -> 0.1
- link tool: mass 1 -> 0.1

Commit message: Drinking and Bed bathing tasks now implemented in v1.0.

File: assistive_gym/envs/assets/bed_bathing/wiper.urdf (robot description, URDF)
Before this commit: robot wiper, 3 links, 2 joints
Links:
- link cloth: geometry collision box size=0.09 0.04 0.005; visual box size=0.09 0.04 0.005
Joints:
- joint j_weld1: origin xyz=0 0 -0.0075 -> xyz=0 0 -0.004
