Commit message: Implemented and tested Stretch robot for itch scratching, bed bathing, and dressing. Fixed control and friction issues for robots with drivable bases, such as the Stretch. Fixed an error with active human environments that prevented the humans from moving.

File: assistive_gym/envs/assets/stretch/stretch_uncalibrated.urdf (robot description, URDF)
Before this commit: robot stretch_description, 37 links, 36 joints
Joints:
- joint joint_left_wheel: origin xyz=-0.00300000000001899 0.15765 0.0507999999999994 rpy=-1.5707963267949 3.16227047920818E-31 7.88745438253713E-16 -> xyz=-0.003 0.15765 0.0508 rpy=-1.5707963267949 3.16227047920818E-31 7.88745438253713E-16
- joint joint_right_wheel: origin xyz=-0.00300000000000034 -0.15765 0.0508000000000004 rpy=-1.57079632679489 -1.11022302462516E-16 7.28583859910277E-17 -> xyz=-0.003 -0.15765 0.0508 rpy=-1.57079632679489 -1.11022302462516E-16 7.28583859910277E-17
