Commit message: Beginning tessts of SMPL-X human mesh implemented in Assistive Gym

File: assistive_gym/envs/assets/wheelchair2/wheelchair.urdf (robot description, URDF)
Before this commit: robot bed, 1 links, 0 joints
Links:
- link root: geometry collision mesh filename=wheelchair_new_compressed_vhacd.obj scale=0.36 0.28 0.36; visual mesh filename=wheelchair_new_compressed.obj scale=0.36 0.28 0.36
