Commit message: Update to wheelchair link for wheeelchair-mounted robots

File: assistive_gym/envs/assets/wheelchair/wheelchair_jaco.urdf (robot description, URDF)
Before this commit: robot wheelchair, 3 links, 2 joints
Joints:
- joint wheelchair_joint: origin xyz=0 0 0 -> xyz=0 0 0 rpy=1.57079632679 0 3.14159265359
- joint wheelchair_joint2: origin xyz=0 0 0 -> xyz=0 0 0 rpy=1.57079632679 0 3.14159265359

File: assistive_gym/envs/assets/wheelchair/wheelchair_jaco_left.urdf (robot description, URDF)
Before this commit: robot wheelchair, 3 links, 2 joints
Joints:
- joint wheelchair_joint: origin xyz=0 0 0 -> xyz=0 0 0 rpy=1.57079632679 0 3.14159265359
- joint wheelchair_joint2: origin xyz=0 0 0 -> xyz=0 0 0 rpy=1.57079632679 0 3.14159265359

Commit message: Significant speed up to initialize and optimize a robot starting pose. Added new figures and feature list for v1.0.

File: assistive_gym/envs/assets/wheelchair/wheelchair_jaco.urdf (robot description, URDF)
Before this commit: robot wheelchair, 3 links, 2 joints
Links:
- link wheelchair_link: geometry visual cylinder length=0.4 radius=0.0425
- link wheelchair_link2: geometry visual cylinder length=0.4 radius=0.0425

File: assistive_gym/envs/assets/wheelchair/wheelchair_jaco_left.urdf (robot description, URDF)
Before this commit: robot wheelchair, 3 links, 2 joints
Links:
- link wheelchair_link: geometry visual cylinder length=0.4 radius=0.0425
- link wheelchair_link2: geometry visual cylinder length=0.4 radius=0.0425
