Commit message: New function for converting obj to agent. Improved Panda robot initial poses

File: assistive_gym/envs/assets/panda/panda.urdf (robot description, URDF)
Before this commit: robot panda, 12 links, 11 joints
Links:
- added link panda_fingercenter
Joints:
- added joint panda_fingercenter_joint: type fixed, parent panda_hand, child panda_fingercenter, origin xyz=0 0 0.1025 rpy=0 0 0, axis 0 0 0

Commit message: Support for Python 3.7, fix for Google Colab (which now uses 3.7), and improved joint angle initialization for the Panda robot

File: assistive_gym/envs/assets/panda/panda.urdf (robot description, URDF)
Before this commit: robot panda, 13 links, 12 joints
Links:
- link panda_fingercenter: mass None -> 0
- link panda_hand: mass None -> 0.73
- link panda_leftfinger: mass None -> 0.1
- link panda_link0: mass None -> 2.92
- link panda_link1: mass None -> 2.74
- link panda_link2: mass None -> 2.74
- link panda_link3: mass None -> 2.38
- link panda_link4: mass None -> 2.38
- link panda_link5: mass None -> 2.74
- link panda_link6: mass None -> 1.55
- link panda_link7: mass None -> 0.54
- link panda_link8: mass None -> 0
- link panda_rightfinger: mass None -> 0.1
