Commit message: fix global orient. debug and fix model flyaway (trick is just dont let body penetrade the floor and set contact damping high enough

File: test_mesh_bk.urdf (robot description, URDF)
Before this commit: robot human, 94 links, 93 joints
Links:
- link head_limb: mass 2.00000 -> 4.92798
- link left_ankle_limb: mass 2.00000 -> 0.72933
- link left_clavicle_limb: mass 2.00000 -> 1.37432
- link left_elbow_limb: mass 2.00000 -> 1.26012
- link left_foot_limb: mass 2.00000 -> 0.15744
- link left_hand_limb: mass 2.00000 -> 0.18707
- link left_hip_limb: mass 2.00000 -> 9.34228
- link left_knee_limb: mass 2.00000 -> 3.94732
- link left_lowarm_limb: mass 2.00000 -> 0.34808
- link left_shoulder_limb: mass 2.00000 -> 2.13791
- link neck_limb: mass 2.00000 -> 0.73358
- link pelvis_limb: mass 2.00000 -> 20.22704
- link right_ankle_limb: mass 2.00000 -> 0.74510
- link right_clavicle_limb: mass 2.00000 -> 1.31272
- link right_elbow_limb: mass 2.00000 -> 1.29671
- link right_foot_limb: mass 2.00000 -> 0.18172
- link right_hand_limb: mass 2.00000 -> 0.19712
- link right_hip_limb: mass 2.00000 -> 8.96915
- link right_knee_limb: mass 2.00000 -> 3.89324
- link right_lowarm_limb: mass 2.00000 -> 0.37314
- link right_shoulder_limb: mass 2.00000 -> 2.29994
- link spine_2_limb: mass 2.00000 -> 8.60388
- link spine_3_limb: mass 2.00000 -> 7.43187
- link spine_4_limb: mass 2.00000 -> 16.44672
Joints:
- joint head_rx: limit lower=-3.14 upper=3.14 effort=1000.00000 velocity=0.00000 -> lower=-0.52360 upper=0.52360 effort=1000.00000 velocity=0.00000; origin xyz=0.01011 0.08894 0.05041 rpy=0.00000 0.0000 0.00000 -> xyz=0.01030 0.08824 0.05158 rpy=0.00000 -0.00000 0.00000
- joint head_ry: limit lower=-3.14 upper=3.14 effort=1000.00000 velocity=0.00000 -> lower=-0.08727 upper=0.08727 effort=1000.00000 velocity=0.00000; origin xyz=0.00000 0.00000 0.00000 rpy=0.00000 0.0000 0.00000 -> xyz=0.00000 0.00000 0.00000 rpy=0.00000 -0.00000 0.00000
- joint head_rz: limit lower=-3.14 upper=3.14 effort=1000.00000 velocity=0.00000 -> lower=-0.08727 upper=0.08727 effort=1000.00000 velocity=0.00000; origin xyz=0.00000 0.00000 0.00000 rpy=0.00000 0.0000 0.00000 -> xyz=0.00000 0.00000 0.00000 rpy=0.00000 -0.00000 0.00000
- joint head_rzdammy: axis (none) -> 0.00000 0.00000 0.00000; origin xyz=0.00000 0.00000 0.00000 rpy=0.00000 0.0000 0.00000 -> xyz=0.00000 0.00000 0.00000 rpy=0.00000 -0.00000 0.00000
- joint left_ankle_rx: limit lower=-3.14 upper=3.14 effort=1000.00000 velocity=0.00000 -> lower=-0.52360 upper=0.52360 effort=1000.00000 velocity=0.00000; origin xyz=-0.01479 -0.42687 -0.03743 rpy=0.00000 0.0000 0.00000 -> xyz=-0.01575 -0.42194 -0.03980 rpy=0.00000 -0.00000 0.00000
- joint left_ankle_ry: limit lower=-3.14 upper=3.14 effort=1000.00000 velocity=0.00000 -> lower=-0.52360 upper=0.52360 effort=1000.00000 velocity=0.00000; origin xyz=0.00000 0.00000 0.00000 rpy=0.00000 0.0000 0.00000 -> xyz=0.00000 0.00000 0.00000 rpy=0.00000 -0.00000 0.00000
- joint left_ankle_rz: limit lower=-3.14 upper=3.14 effort=1000.00000 velocity=0.00000 -> lower=-0.52360 upper=0.52360 effort=1000.00000 velocity=0.00000; origin xyz=0.00000 0.00000 0.00000 rpy=0.00000 0.0000 0.00000 -> xyz=0.00000 0.00000 0.00000 rpy=0.00000 -0.00000 0.00000
- joint left_ankle_rzdammy: axis (none) -> 0.00000 0.00000 0.00000; origin xyz=0.00000 0.00000 0.00000 rpy=0.00000 0.0000 0.00000 -> xyz=0.00000 0.00000 0.00000 rpy=0.00000 -0.00000 0.00000
- joint left_clavicle_rx: limit lower=-3.14 upper=3.14 effort=1000.00000 velocity=0.00000 -> lower=-0.51720 upper=0.47357 effort=1000.00000 velocity=0.00000; origin xyz=0.07170 0.11400 -0.01890 rpy=0.00000 0.0000 0.00000 -> xyz=0.07379 0.11698 -0.01947 rpy=0.00000 -0.00000 0.00000
- joint left_clavicle_ry: limit lower=-3.14 upper=3.14 effort=1000.00000 velocity=0.00000 -> lower=-0.81856 upper=0.25424 effort=1000.00000 velocity=0.00000; origin xyz=0.00000 0.00000 0.00000 rpy=0.00000 0.0000 0.00000 -> xyz=0.00000 0.00000 0.00000 rpy=0.00000 -0.00000 0.00000
- joint left_clavicle_rz: limit lower=-3.14 upper=3.14 effort=1000.00000 velocity=0.00000 -> lower=-0.52360 upper=0.46775 effort=1000.00000 velocity=0.00000; origin xyz=0.00000 0.00000 0.00000 rpy=0.00000 0.0000 0.00000 -> xyz=0.00000 0.00000 0.00000 rpy=0.00000 -0.00000 0.00000
- joint left_clavicle_rzdammy: axis (none) -> 0.00000 0.00000 0.00000; origin xyz=0.00000 0.00000 0.00000 rpy=0.00000 0.0000 0.00000 -> xyz=0.00000 0.00000 0.00000 rpy=0.00000 -0.00000 0.00000
- joint left_elbow_rx: limit lower=-3.14 upper=3.14 effort=1000.00000 velocity=0.00000 -> lower=-2.57087 upper=0.04887 effort=1000.00000 velocity=0.00000; origin xyz=0.25533 -0.01565 -0.02295 rpy=0.00000 0.0000 0.00000 -> xyz=0.25051 -0.01453 -0.02443 rpy=0.00000 -0.00000 0.00000
- joint left_elbow_ry: limit lower=-3.14 upper=3.14 effort=1000.00000 velocity=0.00000 -> lower=0.00000 upper=0.00000 effort=1000.00000 velocity=0.00000; origin xyz=0.00000 0.00000 0.00000 rpy=0.00000 0.0000 0.00000 -> xyz=0.00000 0.00000 0.00000 rpy=0.00000 -0.00000 0.00000
- joint left_elbow_rz: limit lower=-3.14 upper=3.14 effort=1000.00000 velocity=0.00000 -> lower=0.00000 upper=0.00000 effort=1000.00000 velocity=0.00000; origin xyz=0.00000 0.00000 0.00000 rpy=0.00000 0.0000 0.00000 -> xyz=0.00000 0.00000 0.00000 rpy=0.00000 -0.00000 0.00000
- joint left_elbow_rzdammy: axis (none) -> 0.00000 0.00000 0.00000; origin xyz=0.00000 0.00000 0.00000 rpy=0.00000 0.0000 0.00000 -> xyz=0.00000 0.00000 0.00000 rpy=0.00000 -0.00000 0.00000
- joint left_foot_rx: limit lower=-3.14 upper=3.14 effort=1000.00000 velocity=0.00000 -> lower=-0.52360 upper=0.52360 effort=1000.00000 velocity=0.00000; origin xyz=0.04105 -0.06029 0.12204 rpy=0.00000 0.0000 0.00000 -> xyz=0.03813 -0.05994 0.12314 rpy=0.00000 -0.00000 0.00000
- joint left_foot_ry: limit lower=-3.14 upper=3.14 effort=1000.00000 velocity=0.00000 -> lower=-0.52360 upper=0.52360 effort=1000.00000 velocity=0.00000; origin xyz=0.00000 0.00000 0.00000 rpy=0.00000 0.0000 0.00000 -> xyz=0.00000 0.00000 0.00000 rpy=0.00000 -0.00000 0.00000
- joint left_foot_rz: limit lower=-3.14 upper=3.14 effort=0.00000 velocity=0.00000 -> lower=-0.52360 upper=0.52360 effort=0.00000 velocity=0.00000; origin xyz=0.00000 0.00000 0.00000 rpy=0.00000 0.0000 0.00000 -> xyz=0.00000 0.00000 0.00000 rpy=0.00000 -0.00000 0.00000
- joint left_foot_rzdammy: axis (none) -> 0.00000 0.00000 0.00000; origin xyz=0.00000 0.00000 0.00000 rpy=0.00000 0.0000 0.00000 -> xyz=0.00000 0.00000 0.00000 rpy=0.00000 -0.00000 0.00000
- joint left_hand_rx: limit lower=-3.14 upper=3.14 effort=1000.00000 velocity=0.00000 -> lower=-0.52360 upper=0.52360 effort=1000.00000 velocity=0.00000; origin xyz=0.08669 -0.01064 -0.01559 rpy=0.00000 0.0000 0.00000 -> xyz=0.08704 -0.01083 -0.01551 rpy=0.00000 -0.00000 0.00000
- joint left_hand_ry: limit lower=-3.14 upper=3.14 effort=1000.00000 velocity=0.00000 -> lower=-0.52360 upper=0.52360 effort=1000.00000 velocity=0.00000; origin xyz=0.00000 0.00000 0.00000 rpy=0.00000 0.0000 0.00000 -> xyz=0.00000 0.00000 0.00000 rpy=0.00000 -0.00000 0.00000
- joint left_hand_rz: limit lower=-3.14 upper=3.14 effort=1000.00000 velocity=0.00000 -> lower=-0.52360 upper=0.52360 effort=1000.00000 velocity=0.00000; origin xyz=0.00000 0.00000 0.00000 rpy=0.00000 0.0000 0.00000 -> xyz=0.00000 0.00000 0.00000 rpy=0.00000 -0.00000 0.00000
- joint left_hand_rzdammy: axis (none) -> 0.00000 0.00000 0.00000; origin xyz=0.00000 0.00000 0.00000 rpy=0.00000 0.0000 0.00000 -> xyz=0.00000 0.00000 0.00000 rpy=0.00000 -0.00000 0.00000
- joint left_hip_rx: limit lower=-3.14 upper=3.14 effort=1000.00000 velocity=0.00000 -> lower=-1.57080 upper=0.31067 effort=1000.00000 velocity=0.00000; origin xyz=0.05858 -0.08228 -0.01766 rpy=0.00000 0.0000 0.00000 -> xyz=0.06231 -0.08478 -0.01632 rpy=0.00000 -0.00000 0.00000
- joint left_hip_ry: limit lower=-3.14 upper=3.14 effort=1000.00000 velocity=0.00000 -> lower=-0.58818 upper=0.56898 effort=1000.00000 velocity=0.00000; origin xyz=0.00000 0.00000 0.00000 rpy=0.00000 0.0000 0.00000 -> xyz=0.00000 0.00000 0.00000 rpy=0.00000 -0.00000 0.00000
- joint left_hip_rz: limit lower=-3.14 upper=3.14 effort=1000.00000 velocity=0.00000 -> lower=-0.53233 upper=0.67370 effort=1000.00000 velocity=0.00000; origin xyz=0.00000 0.00000 0.00000 rpy=0.00000 0.0000 0.00000 -> xyz=0.00000 0.00000 0.00000 rpy=0.00000 -0.00000 0.00000
- joint left_hip_rzdammy: axis (none) -> 0.00000 0.00000 0.00000; origin xyz=0.00000 0.00000 0.00000 rpy=0.00000 0.0000 0.00000 -> xyz=0.00000 0.00000 0.00000 rpy=0.00000 -0.00000 0.00000
- joint left_knee_rx: limit lower=-3.14 upper=3.14 effort=1000.00000 velocity=0.00000 -> lower=-0.02269 upper=2.44172 effort=1000.00000 velocity=0.00000; origin xyz=0.04345 -0.38647 0.00804 rpy=0.00000 0.0000 0.00000 -> xyz=0.04098 -0.37890 0.00622 rpy=0.00000 -0.00000 0.00000
- joint left_knee_ry: limit lower=-3.14 upper=3.14 effort=1000.00000 velocity=0.00000 -> lower=0.00000 upper=0.00000 effort=1000.00000 velocity=0.00000; origin xyz=0.00000 0.00000 0.00000 rpy=0.00000 0.0000 0.00000 -> xyz=0.00000 0.00000 0.00000 rpy=0.00000 -0.00000 0.00000
- joint left_knee_rz: limit lower=-3.14 upper=3.14 effort=1000.00000 velocity=0.00000 -> lower=0.00000 upper=0.00000 effort=1000.00000 velocity=0.00000; origin xyz=0.00000 0.00000 0.00000 rpy=0.00000 0.0000 0.00000 -> xyz=0.00000 0.00000 0.00000 rpy=0.00000 -0.00000 0.00000
- joint left_knee_rzdammy: origin xyz=0.00000 0.00000 0.00000 rpy=0.00000 0.0000 0.00000 -> xyz=0.00000 0.00000 0.00000 rpy=0.00000 -0.00000 0.00000
- joint left_lowarm_rx: limit lower=-3.14 upper=3.14 effort=1000.00000 velocity=0.00000 -> lower=-0.52360 upper=0.52360 effort=1000.00000 velocity=0.00000; origin xyz=0.26571 0.01270 -0.00737 rpy=0.00000 0.0000 0.00000 -> xyz=0.26348 0.01330 -0.00622 rpy=0.00000 -0.00000 0.00000
- joint left_lowarm_ry: limit lower=-3.14 upper=3.14 effort=1000.00000 velocity=0.00000 -> lower=-0.52360 upper=0.52360 effort=1000.00000 velocity=0.00000; origin xyz=0.00000 0.00000 0.00000 rpy=0.00000 0.0000 0.00000 -> xyz=0.00000 0.00000 0.00000 rpy=0.00000 -0.00000 0.00000
- joint left_lowarm_rz: limit lower=-3.14 upper=3.14 effort=1000.00000 velocity=0.00000 -> lower=-0.52360 upper=0.52360 effort=1000.00000 velocity=0.00000; origin xyz=0.00000 0.00000 0.00000 rpy=0.00000 0.0000 0.00000 -> xyz=0.00000 0.00000 0.00000 rpy=0.00000 -0.00000 0.00000
- joint left_lowarm_rzdammy: axis (none) -> 0.00000 0.00000 0.00000; origin xyz=0.00000 0.00000 0.00000 rpy=0.00000 0.0000 0.00000 -> xyz=0.00000 0.00000 0.00000 rpy=0.00000 -0.00000 0.00000
- joint left_shoulder_rx: limit lower=-3.14 upper=3.14 effort=1000.00000 velocity=0.00000 -> lower=-1.03440 upper=0.94713 effort=1000.00000 velocity=0.00000; origin xyz=0.12292 0.04521 -0.01905 rpy=0.00000 0.0000 0.00000 -> xyz=0.12634 0.04464 -0.02146 rpy=0.00000 -0.00000 0.00000
- joint left_shoulder_ry: limit lower=-3.14 upper=3.14 effort=1000.00000 velocity=0.00000 -> lower=-1.63712 upper=0.50847 effort=1000.00000 velocity=0.00000; origin xyz=0.00000 0.00000 0.00000 rpy=0.00000 0.0000 0.00000 -> xyz=0.00000 0.00000 0.00000 rpy=0.00000 -0.00000 0.00000
- joint left_shoulder_rz: limit lower=-3.14 upper=3.14 effort=1000.00000 velocity=0.00000 -> lower=-1.04720 upper=0.93550 effort=1000.00000 velocity=0.00000; origin xyz=0.00000 0.00000 0.00000 rpy=0.00000 0.0000 0.00000 -> xyz=0.00000 0.00000 0.00000 rpy=0.00000 -0.00000 0.00000
- joint left_shoulder_rzdammy: axis (none) -> 0.00000 0.00000 0.00000; origin xyz=0.00000 0.00000 0.00000 rpy=0.00000 0.0000 0.00000 -> xyz=0.00000 0.00000 0.00000 rpy=0.00000 -0.00000 0.00000
- joint neck_rx: limit lower=-3.14 upper=3.14 effort=1000.00000 velocity=0.00000 -> lower=-0.52360 upper=0.52360 effort=1000.00000 velocity=0.00000; origin xyz=-0.01339 0.21164 -0.03347 rpy=0.00000 0.0000 0.00000 -> xyz=-0.01322 0.21753 -0.03787 rpy=0.00000 -0.00000 0.00000
- joint neck_ry: limit lower=-3.14 upper=3.14 effort=1000.00000 velocity=0.00000 -> lower=-0.08727 upper=0.08727 effort=1000.00000 velocity=0.00000; origin xyz=0.00000 0.00000 0.00000 rpy=0.00000 0.0000 0.00000 -> xyz=0.00000 0.00000 0.00000 rpy=0.00000 -0.00000 0.00000
- joint neck_rz: limit lower=-3.14 upper=3.14 effort=1000.00000 velocity=0.00000 -> lower=-0.08727 upper=0.08727 effort=1000.00000 velocity=0.00000; origin xyz=0.00000 0.00000 0.00000 rpy=0.00000 0.0000 0.00000 -> xyz=0.00000 0.00000 0.00000 rpy=0.00000 -0.00000 0.00000
- joint neck_rzdammy: axis (none) -> 0.00000 0.00000 0.00000; origin xyz=0.00000 0.00000 0.00000 rpy=0.00000 0.0000 0.00000 -> xyz=0.00000 0.00000 0.00000 rpy=0.00000 -0.00000 0.00000
- joint pelvis: origin xyz=0.00000 0.00000 0.00000 rpy=0.00000 0.0000 0.00000 -> xyz=0.00000 0.00000 0.00000 rpy=0.00000 -0.00000 0.00000
- joint right_ankle_rx: limit lower=-3.14 upper=3.14 effort=1000.00000 velocity=0.00000 -> lower=-0.52360 upper=0.52360 effort=1000.00000 velocity=0.00000; origin xyz=0.01906 -0.42005 -0.03456 rpy=0.00000 0.0000 0.00000 -> xyz=0.01945 -0.41561 -0.03688 rpy=0.00000 -0.00000 0.00000
- joint right_ankle_ry: limit lower=-3.14 upper=3.14 effort=1000.00000 velocity=0.00000 -> lower=-0.52360 upper=0.52360 effort=1000.00000 velocity=0.00000; origin xyz=0.00000 0.00000 0.00000 rpy=0.00000 0.0000 0.00000 -> xyz=0.00000 0.00000 0.00000 rpy=0.00000 -0.00000 0.00000
- joint right_ankle_rz: limit lower=-3.14 upper=3.14 effort=1000.00000 velocity=0.00000 -> lower=-0.52360 upper=0.52360 effort=1000.00000 velocity=0.00000; origin xyz=0.00000 0.00000 0.00000 rpy=0.00000 0.0000 0.00000 -> xyz=0.00000 0.00000 0.00000 rpy=0.00000 -0.00000 0.00000
- joint right_ankle_rzdammy: axis (none) -> 0.00000 0.00000 0.00000; origin xyz=0.00000 0.00000 0.00000 rpy=0.00000 0.0000 0.00000 -> xyz=0.00000 0.00000 0.00000 rpy=0.00000 -0.00000 0.00000
- joint right_clavicle_rx: limit lower=-3.14 upper=3.14 effort=1000.00000 velocity=0.00000 -> lower=-0.51720 upper=0.47357 effort=1000.00000 velocity=0.00000; origin xyz=-0.08295 0.11247 -0.02371 rpy=0.00000 0.0000 0.00000 -> xyz=-0.08499 0.11515 -0.02500 rpy=0.00000 -0.00000 0.00000
- joint right_clavicle_ry: limit lower=-3.14 upper=3.14 effort=1000.00000 velocity=0.00000 -> lower=-0.25424 upper=0.81856 effort=1000.00000 velocity=0.00000; origin xyz=0.00000 0.00000 0.00000 rpy=0.00000 0.0000 0.00000 -> xyz=0.00000 0.00000 0.00000 rpy=0.00000 -0.00000 0.00000
- joint right_clavicle_rz: limit lower=-3.14 upper=3.14 effort=1000.00000 velocity=0.00000 -> lower=-0.52360 upper=0.46775 effort=1000.00000 velocity=0.00000; origin xyz=0.00000 0.00000 0.00000 rpy=0.00000 0.0000 0.00000 -> xyz=0.00000 0.00000 0.00000 rpy=0.00000 -0.00000 0.00000
- joint right_clavicle_rzdammy: axis (none) -> 0.00000 0.00000 0.00000; origin xyz=0.00000 0.00000 0.00000 rpy=0.00000 0.0000 0.00000 -> xyz=0.00000 0.00000 0.00000 rpy=0.00000 -0.00000 0.00000
- joint right_elbow_rx: limit lower=-3.14 upper=3.14 effort=1000.00000 velocity=0.00000 -> lower=-0.04887 upper=2.57087 effort=1000.00000 velocity=0.00000; origin xyz=-0.26013 -0.01437 -0.03127 rpy=0.00000 0.0000 0.00000 -> xyz=-0.25664 -0.01184 -0.03424 rpy=0.00000 -0.00000 0.00000
- joint right_elbow_ry: limit lower=-3.14 upper=3.14 effort=1000.00000 velocity=0.00000 -> lower=0.00000 upper=0.00000 effort=1000.00000 velocity=0.00000; origin xyz=0.00000 0.00000 0.00000 rpy=0.00000 0.0000 0.00000 -> xyz=0.00000 0.00000 0.00000 rpy=0.00000 -0.00000 0.00000
- joint right_elbow_rz: limit lower=-3.14 upper=3.14 effort=1000.00000 velocity=0.00000 -> lower=0.00000 upper=0.00000 effort=1000.00000 velocity=0.00000; origin xyz=0.00000 0.00000 0.00000 rpy=0.00000 0.0000 0.00000 -> xyz=0.00000 0.00000 0.00000 rpy=0.00000 -0.00000 0.00000
- joint right_elbow_rzdammy: axis (none) -> 0.00000 0.00000 0.00000; origin xyz=0.00000 0.00000 0.00000 rpy=0.00000 0.0000 0.00000 -> xyz=0.00000 0.00000 0.00000 rpy=0.00000 -0.00000 0.00000
- joint right_foot_rx: limit lower=-3.14 upper=3.14 effort=1000.00000 velocity=0.00000 -> lower=-0.52360 upper=0.52360 effort=1000.00000 velocity=0.00000; origin xyz=-0.03484 -0.06211 0.13032 rpy=0.00000 0.0000 0.00000 -> xyz=-0.03638 -0.06116 0.13115 rpy=0.00000 -0.00000 0.00000
- joint right_foot_ry: limit lower=-3.14 upper=3.14 effort=1000.00000 velocity=0.00000 -> lower=-0.52360 upper=0.52360 effort=1000.00000 velocity=0.00000; origin xyz=0.00000 0.00000 0.00000 rpy=0.00000 0.0000 0.00000 -> xyz=0.00000 0.00000 0.00000 rpy=0.00000 -0.00000 0.00000
- joint right_foot_rz: limit lower=-3.14 upper=3.14 effort=1000.00000 velocity=0.00000 -> lower=-0.52360 upper=0.52360 effort=1000.00000 velocity=0.00000; origin xyz=0.00000 0.00000 0.00000 rpy=0.00000 0.0000 0.00000 -> xyz=0.00000 0.00000 0.00000 rpy=0.00000 -0.00000 0.00000
- joint right_foot_rzdammy: axis (none) -> 0.00000 0.00000 0.00000; origin xyz=0.00000 0.00000 0.00000 rpy=0.00000 0.0000 0.00000 -> xyz=0.00000 0.00000 0.00000 rpy=0.00000 -0.00000 0.00000
- joint right_hand_rx: limit lower=-3.14 upper=3.14 effort=1000.00000 velocity=0.00000 -> lower=-0.52360 upper=0.52360 effort=1000.00000 velocity=0.00000; origin xyz=-0.08875 -0.00865 -0.01011 rpy=0.00000 0.0000 0.00000 -> xyz=-0.08935 -0.00882 -0.00999 rpy=0.00000 -0.00000 0.00000
- joint right_hand_ry: limit lower=-3.14 upper=3.14 effort=1000.00000 velocity=0.00000 -> lower=-0.52360 upper=0.52360 effort=1000.00000 velocity=0.00000; origin xyz=0.00000 0.00000 0.00000 rpy=0.00000 0.0000 0.00000 -> xyz=0.00000 0.00000 0.00000 rpy=0.00000 -0.00000 0.00000
- joint right_hand_rz: limit lower=-3.14 upper=3.14 effort=1000.00000 velocity=0.00000 -> lower=-0.52360 upper=0.52360 effort=1000.00000 velocity=0.00000; origin xyz=0.00000 0.00000 0.00000 rpy=0.00000 0.0000 0.00000 -> xyz=0.00000 0.00000 0.00000 rpy=0.00000 -0.00000 0.00000
- joint right_hand_rzdammy: axis (none) -> 0.00000 0.00000 0.00000; origin xyz=0.00000 0.00000 0.00000 rpy=0.00000 0.0000 0.00000 -> xyz=0.00000 0.00000 0.00000 rpy=0.00000 -0.00000 0.00000
- joint right_hip_rx: limit lower=-3.14 upper=3.14 effort=1000.00000 velocity=0.00000 -> lower=-1.57080 upper=0.31067 effort=1000.00000 velocity=0.00000; origin xyz=-0.06031 -0.09051 -0.01354 rpy=0.00000 0.0000 0.00000 -> xyz=-0.06426 -0.09295 -0.01172 rpy=0.00000 -0.00000 0.00000
- joint right_hip_ry: limit lower=-3.14 upper=3.14 effort=1000.00000 velocity=0.00000 -> lower=-0.56898 upper=0.58818 effort=1000.00000 velocity=0.00000; origin xyz=0.00000 0.00000 0.00000 rpy=0.00000 0.0000 0.00000 -> xyz=0.00000 0.00000 0.00000 rpy=0.00000 -0.00000 0.00000
- joint right_hip_rz: limit lower=-3.14 upper=3.14 effort=1000.00000 velocity=0.00000 -> lower=-0.67370 upper=0.53233 effort=1000.00000 velocity=0.00000; origin xyz=0.00000 0.00000 0.00000 rpy=0.00000 0.0000 0.00000 -> xyz=0.00000 0.00000 0.00000 rpy=0.00000 -0.00000 0.00000
- joint right_hip_rzdammy: axis (none) -> 0.00000 0.00000 0.00000; origin xyz=0.00000 0.00000 0.00000 rpy=0.00000 0.0000 0.00000 -> xyz=0.00000 0.00000 0.00000 rpy=0.00000 -0.00000 0.00000
- joint right_knee_rx: limit lower=-3.14 upper=3.14 effort=1000.00000 velocity=0.00000 -> lower=-0.02269 upper=2.44172 effort=1000.00000 velocity=0.00000; origin xyz=-0.04326 -0.38369 -0.00484 rpy=0.00000 0.0000 0.00000 -> xyz=-0.04112 -0.37826 -0.00642 rpy=0.00000 -0.00000 0.00000
- joint right_knee_ry: limit lower=-3.14 upper=3.14 effort=1000.00000 velocity=0.00000 -> lower=0.00000 upper=0.00000 effort=1000.00000 velocity=0.00000; origin xyz=0.00000 0.00000 0.00000 rpy=0.00000 0.0000 0.00000 -> xyz=0.00000 0.00000 0.00000 rpy=0.00000 -0.00000 0.00000
- joint right_knee_rz: limit lower=-3.14 upper=3.14 effort=1000.00000 velocity=0.00000 -> lower=0.00000 upper=0.00000 effort=1000.00000 velocity=0.00000; origin xyz=0.00000 0.00000 0.00000 rpy=0.00000 0.0000 0.00000 -> xyz=0.00000 0.00000 0.00000 rpy=0.00000 -0.00000 0.00000
- joint right_knee_rzdammy: axis (none) -> 0.00000 0.00000 0.00000; origin xyz=0.00000 0.00000 0.00000 rpy=0.00000 0.0000 0.00000 -> xyz=0.00000 0.00000 0.00000 rpy=0.00000 -0.00000 0.00000
- joint right_lowarm_rx: limit lower=-3.14 upper=3.14 effort=1000.00000 velocity=0.00000 -> lower=-0.52360 upper=0.52360 effort=1000.00000 velocity=0.00000; origin xyz=-0.26911 0.00679 -0.00603 rpy=0.00000 0.0000 0.00000 -> xyz=-0.26554 0.00531 -0.00574 rpy=0.00000 -0.00000 0.00000
- joint right_lowarm_ry: limit lower=-3.14 upper=3.14 effort=1000.00000 velocity=0.00000 -> lower=-0.52360 upper=0.52360 effort=1000.00000 velocity=0.00000; origin xyz=0.00000 0.00000 0.00000 rpy=0.00000 0.0000 0.00000 -> xyz=0.00000 0.00000 0.00000 rpy=0.00000 -0.00000 0.00000
- joint right_lowarm_rz: limit lower=-3.14 upper=3.14 effort=1000.00000 velocity=0.00000 -> lower=-0.52360 upper=0.52360 effort=1000.00000 velocity=0.00000; origin xyz=0.00000 0.00000 0.00000 rpy=0.00000 0.0000 0.00000 -> xyz=0.00000 0.00000 0.00000 rpy=0.00000 -0.00000 0.00000
- joint right_lowarm_rzdammy: axis (none) -> 0.00000 0.00000 0.00000; origin xyz=0.00000 0.00000 0.00000 rpy=0.00000 0.0000 0.00000 -> xyz=0.00000 0.00000 0.00000 rpy=0.00000 -0.00000 0.00000
- joint right_shoulder_rx: limit lower=-3.14 upper=3.14 effort=1000.00000 velocity=0.00000 -> lower=-1.03440 upper=0.94713 effort=1000.00000 velocity=0.00000; origin xyz=-0.11323 0.04685 -0.00847 rpy=0.00000 0.0000 0.00000 -> xyz=-0.11654 0.04630 -0.01035 rpy=0.00000 -0.00000 0.00000
- joint right_shoulder_ry: limit lower=-3.14 upper=3.14 effort=1000.00000 velocity=0.00000 -> lower=-0.50847 upper=1.63712 effort=1000.00000 velocity=0.00000; origin xyz=0.00000 0.00000 0.00000 rpy=0.00000 0.0000 0.00000 -> xyz=0.00000 0.00000 0.00000 rpy=0.00000 -0.00000 0.00000
- joint right_shoulder_rz: limit lower=-3.14 upper=3.14 effort=1000.00000 velocity=0.00000 -> lower=-1.04720 upper=0.93550 effort=1000.00000 velocity=0.00000; origin xyz=0.00000 0.00000 0.00000 rpy=0.00000 0.0000 0.00000 -> xyz=0.00000 0.00000 0.00000 rpy=0.00000 -0.00000 0.00000
- joint right_shoulder_rzdammy: axis (none) -> 0.00000 0.00000 0.00000; origin xyz=0.00000 0.00000 0.00000 rpy=0.00000 0.0000 0.00000 -> xyz=0.00000 0.00000 0.00000 rpy=0.00000 -0.00000 0.00000
- joint spine_2_rx: limit lower=-3.14 upper=3.14 effort=1000.00000 velocity=0.00000 -> lower=-0.52360 upper=0.52360 effort=1000.00000 velocity=0.00000; origin xyz=0.00444 0.12440 -0.03839 rpy=0.00000 0.0000 0.00000 -> xyz=0.00444 0.12916 -0.04297 rpy=0.00000 -0.00000 0.00000
- joint spine_2_ry: limit lower=-3.14 upper=3.14 effort=1000.00000 velocity=0.00000 -> lower=-0.52360 upper=0.52360 effort=1000.00000 velocity=0.00000; origin xyz=0.00000 0.00000 0.00000 rpy=0.00000 0.0000 0.00000 -> xyz=0.00000 0.00000 0.00000 rpy=0.00000 -0.00000 0.00000
- joint spine_2_rz: limit lower=-3.14 upper=3.14 effort=1000.00000 velocity=0.00000 -> lower=-0.52360 upper=0.52360 effort=1000.00000 velocity=0.00000; origin xyz=0.00000 0.00000 0.00000 rpy=0.00000 0.0000 0.00000 -> xyz=0.00000 0.00000 0.00000 rpy=0.00000 -0.00000 0.00000
- joint spine_2_rzdammy: axis (none) -> 0.00000 0.00000 0.00000; origin xyz=0.00000 0.00000 0.00000 rpy=0.00000 0.0000 0.00000 -> xyz=0.00000 0.00000 0.00000 rpy=0.00000 -0.00000 0.00000
- joint spine_3_rx: limit lower=-3.14 upper=3.14 effort=1000.00000 velocity=0.00000 -> lower=-0.52360 upper=0.52360 effort=1000.00000 velocity=0.00000; origin xyz=0.00449 0.13796 0.02682 rpy=0.00000 0.0000 0.00000 -> xyz=0.00482 0.14331 0.02729 rpy=0.00000 -0.00000 0.00000
- joint spine_3_ry: limit lower=-3.14 upper=3.14 effort=1000.00000 velocity=0.00000 -> lower=-0.52360 upper=0.52360 effort=1000.00000 velocity=0.00000; origin xyz=0.00000 0.00000 0.00000 rpy=0.00000 0.0000 0.00000 -> xyz=0.00000 0.00000 0.00000 rpy=0.00000 -0.00000 0.00000
- joint spine_3_rz: limit lower=-3.14 upper=3.14 effort=1000.00000 velocity=0.00000 -> lower=-0.52360 upper=0.52360 effort=1000.00000 velocity=0.00000; origin xyz=0.00000 0.00000 0.00000 rpy=0.00000 0.0000 0.00000 -> xyz=0.00000 0.00000 0.00000 rpy=0.00000 -0.00000 0.00000
- joint spine_3_rzdammy: axis (none) -> 0.00000 0.00000 0.00000; origin xyz=0.00000 0.00000 0.00000 rpy=0.00000 0.0000 0.00000 -> xyz=0.00000 0.00000 0.00000 rpy=0.00000 -0.00000 0.00000
- joint spine_4_rx: limit lower=-3.14 upper=3.14 effort=1000.00000 velocity=0.00000 -> lower=-0.52360 upper=0.52360 effort=1000.00000 velocity=0.00000; origin xyz=-0.00226 0.05603 0.00286 rpy=0.00000 0.0000 0.00000 -> xyz=-0.00247 0.05844 0.00433 rpy=0.00000 -0.00000 0.00000
- joint spine_4_ry: limit lower=-3.14 upper=3.14 effort=1000.00000 velocity=0.00000 -> lower=-0.52360 upper=0.52360 effort=1000.00000 velocity=0.00000; origin xyz=0.00000 0.00000 0.00000 rpy=0.00000 0.0000 0.00000 -> xyz=0.00000 0.00000 0.00000 rpy=0.00000 -0.00000 0.00000
- joint spine_4_rz: limit lower=-3.14 upper=3.14 effort=1000.00000 velocity=0.00000 -> lower=-0.52360 upper=0.52360 effort=1000.00000 velocity=0.00000; origin xyz=0.00000 0.00000 0.00000 rpy=0.00000 0.0000 0.00000 -> xyz=0.00000 0.00000 0.00000 rpy=0.00000 -0.00000 0.00000
- joint spine_4_rzdammy: axis (none) -> 0.00000 0.00000 0.00000; origin xyz=0.00000 0.00000 0.00000 rpy=0.00000 0.0000 0.00000 -> xyz=0.00000 0.00000 0.00000 rpy=0.00000 -0.00000 0.00000
