Commit message: reset meshes and urdf to main

File: test_mesh.urdf (robot description, URDF)
Before this commit: robot human, 94 links, 93 joints
Links:
- link head_limb: geometry collision mesh filename=././././assistive_gym/envs/assets/human/meshes/Head.obj scale=1.00000 1.00000 1.00000; visual mesh filename=././././assistive_gym/envs/assets/human/meshes/Head.obj scale=1.00000 1.00000 1.00000
- link left_ankle_limb: geometry collision mesh filename=././././assistive_gym/envs/assets/human/meshes/L_Ankle.obj scale=1.00000 1.00000 1.00000; visual mesh filename=././././assistive_gym/envs/assets/human/meshes/L_Ankle.obj scale=1.00000 1.00000 1.00000
- link left_clavicle_limb: geometry collision mesh filename=././././assistive_gym/envs/assets/human/meshes/L_Collar.obj scale=1.00000 1.00000 1.00000; visual mesh filename=././././assistive_gym/envs/assets/human/meshes/L_Collar.obj scale=1.00000 1.00000 1.00000
- link left_elbow_limb: geometry collision mesh filename=././././assistive_gym/envs/assets/human/meshes/L_Elbow.obj scale=1.00000 1.00000 1.00000; visual mesh filename=././././assistive_gym/envs/assets/human/meshes/L_Elbow.obj scale=1.00000 1.00000 1.00000
- link left_foot_limb: geometry collision mesh filename=././././assistive_gym/envs/assets/human/meshes/L_Foot.obj scale=1.00000 1.00000 1.00000; visual mesh filename=././././assistive_gym/envs/assets/human/meshes/L_Foot.obj scale=1.00000 1.00000 1.00000
- link left_hand_limb: geometry collision mesh filename=././././assistive_gym/envs/assets/human/meshes/L_Hand.obj scale=1.00000 1.00000 1.00000; visual mesh filename=././././assistive_gym/envs/assets/human/meshes/L_Hand.obj scale=1.00000 1.00000 1.00000
- link left_hip_limb: geometry collision mesh filename=././././assistive_gym/envs/assets/human/meshes/L_Hip.obj scale=1.00000 1.00000 1.00000; visual mesh filename=././././assistive_gym/envs/assets/human/meshes/L_Hip.obj scale=1.00000 1.00000 1.00000
- link left_knee_limb: geometry collision mesh filename=././././assistive_gym/envs/assets/human/meshes/L_Knee.obj scale=1.00000 1.00000 1.00000; visual mesh filename=././././assistive_gym/envs/assets/human/meshes/L_Knee.obj scale=1.00000 1.00000 1.00000
- link left_lowarm_limb: geometry collision mesh filename=././././assistive_gym/envs/assets/human/meshes/L_Wrist.obj scale=1.00000 1.00000 1.00000; visual mesh filename=././././assistive_gym/envs/assets/human/meshes/L_Wrist.obj scale=1.00000 1.00000 1.00000
- link left_shoulder_limb: geometry collision mesh filename=././././assistive_gym/envs/assets/human/meshes/L_Shoulder.o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 scale=1.00000 1.00000 1.00000; visual mesh filename=././././assistive_gym/envs/assets/human/meshes/L_Shoulder.o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 scale=1.00000 1.00000 1.00000
- link neck_limb: geometry collision mesh filename=././././assistive_gym/envs/assets/human/meshes/Neck.obj scale=1.00000 1.00000 1.00000; visual mesh filename=././././assistive_gym/envs/assets/human/meshes/Neck.obj scale=1.00000 1.00000 1.00000
- link pelvis_limb: geometry collision mesh filename=././assistive_gym/envs/assets/human/meshes/Pelvis.obj scale=1.00000 1.00000 1.00000; visual mesh filename=././assistive_gym/envs/assets/human/meshes/Pelvis.obj scale=1.00000 1.00000 1.00000
- link right_ankle_limb: geometry collision mesh filename=././././assistive_gym/envs/assets/human/meshes/R_Ankle.obj scale=1.00000 1.00000 1.00000; visual mesh filename=././././assistive_gym/envs/assets/human/meshes/R_Ankle.obj scale=1.00000 1.00000 1.00000
- link right_clavicle_limb: geometry collision mesh filename=././././assistive_gym/envs/assets/human/meshes/R_Collar.obj scale=1.00000 1.00000 1.00000; visual mesh filename=././././assistive_gym/envs/assets/human/meshes/R_Collar.obj scale=1.00000 1.00000 1.00000
- link right_elbow_limb: geometry collision mesh filename=././././assistive_gym/envs/assets/human/meshes/R_Elbow.obj scale=1.00000 1.00000 1.00000; visual mesh filename=././././assistive_gym/envs/assets/human/meshes/R_Elbow.obj scale=1.00000 1.00000 1.00000
- link right_foot_limb: geometry collision mesh filename=././././assistive_gym/envs/assets/human/meshes/R_Foot.obj scale=1.00000 1.00000 1.00000; visual mesh filename=././././assistive_gym/envs/assets/human/meshes/R_Foot.obj scale=1.00000 1.00000 1.00000
- link right_hand_limb: geometry collision mesh filename=././././assistive_gym/envs/assets/human/meshes/R_Hand.obj scale=1.00000 1.00000 1.00000; visual mesh filename=././././assistive_gym/envs/assets/human/meshes/R_Hand.obj scale=1.00000 1.00000 1.00000
- link right_hip_limb: geometry collision mesh filename=././././assistive_gym/envs/assets/human/meshes/R_Hip.obj scale=1.00000 1.00000 1.00000; visual mesh filename=././././assistive_gym/envs/assets/human/meshes/R_Hip.obj scale=1.00000 1.00000 1.00000
- link right_knee_limb: geometry collision mesh filename=././././assistive_gym/envs/assets/human/meshes/R_Knee.obj scale=1.00000 1.00000 1.00000; visual mesh filename=././././assistive_gym/envs/assets/human/meshes/R_Knee.obj scale=1.00000 1.00000 1.00000
- link right_lowarm_limb: geometry collision mesh filename=././././assistive_gym/envs/assets/human/meshes/R_Wrist.obj scale=1.00000 1.00000 1.00000; visual mesh filename=././././assistive_gym/envs/assets/human/meshes/R_Wrist.obj scale=1.00000 1.00000 1.00000
- link right_shoulder_limb: geometry collision mesh filename=././././assistive_gym/envs/assets/human/meshes/R_Shoulder.o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 scale=1.00000 1.00000 1.00000; visual mesh filename=././././assistive_gym/envs/assets/human/meshes/R_Shoulder.o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 scale=1.00000 1.00000 1.00000
- link spine_2_limb: geometry collision mesh filename=././././assistive_gym/envs/assets/human/meshes/Spine1.obj scale=1.00000 1.00000 1.00000; visual mesh filename=././././assistive_gym/envs/assets/human/meshes/Spine1.obj scale=1.00000 1.00000 1.00000
- link spine_3_limb: geometry collision mesh filename=././././assistive_gym/envs/assets/human/meshes/Spine2.obj scale=1.00000 1.00000 1.00000; visual mesh filename=././././assistive_gym/envs/assets/human/meshes/Spine2.obj scale=1.00000 1.00000 1.00000
- link spine_4_limb: geometry collision mesh filename=././././assistive_gym/envs/assets/human/meshes/Spine3.obj scale=1.00000 1.00000 1.00000; visual mesh filename=././././assistive_gym/envs/assets/human/meshes/Spine3.obj scale=1.00000 1.00000 1.00000
Joints:
- joint head_rx: limit lower=-0.52360 upper=0.52360 effort=1000.00000 velocity=0.00000 -> lower=-3.14000 upper=3.14000 effort=100.0 velocity=1.00000
- joint head_ry: limit lower=-0.08727 upper=0.08727 effort=1000.00000 velocity=0.00000 -> lower=-3.14000 upper=3.14000 effort=100.0 velocity=1.00000
- joint head_rz: limit lower=-0.08727 upper=0.08727 effort=1000.00000 velocity=0.00000 -> lower=-3.14000 upper=3.14000 effort=100.0 velocity=1.00000
- joint left_ankle_rx: limit lower=-0.52360 upper=0.52360 effort=1000.00000 velocity=0.00000 -> lower=-3.14000 upper=3.14000 effort=100.0 velocity=1.00000
- joint left_ankle_ry: limit lower=-0.52360 upper=0.52360 effort=1000.00000 velocity=0.00000 -> lower=-3.14000 upper=3.14000 effort=100.0 velocity=1.00000
- joint left_ankle_rz: limit lower=-0.52360 upper=0.52360 effort=1000.00000 velocity=0.00000 -> lower=-3.14000 upper=3.14000 effort=100.0 velocity=1.00000
- joint left_clavicle_rx: limit lower=-0.51720 upper=0.47357 effort=1000.00000 velocity=0.00000 -> lower=-3.14000 upper=3.14000 effort=100.0 velocity=1.00000
- joint left_clavicle_ry: limit lower=-0.81856 upper=0.25424 effort=1000.00000 velocity=0.00000 -> lower=-3.14000 upper=3.14000 effort=100.0 velocity=1.00000
- joint left_clavicle_rz: limit lower=-0.52360 upper=0.46775 effort=1000.00000 velocity=0.00000 -> lower=-3.14000 upper=3.14000 effort=100.0 velocity=1.00000
- joint left_elbow_rx: limit lower=0.00000 upper=0.00000 effort=1000.00000 velocity=0.00000 -> lower=-3.14000 upper=3.14000 effort=100.0 velocity=1.00000
- joint left_elbow_ry: limit lower=-2.57087 upper=0.04887 effort=1000.00000 velocity=0.00000 -> lower=-3.14000 upper=3.14000 effort=100.0 velocity=1.00000
- joint left_elbow_rz: limit lower=0.00000 upper=0.00000 effort=1000.00000 velocity=0.00000 -> lower=-3.14000 upper=3.14000 effort=100.0 velocity=1.00000
- joint left_foot_rx: limit lower=-0.52360 upper=0.52360 effort=1000.00000 velocity=0.00000 -> lower=-3.14000 upper=3.14000 effort=100.0 velocity=1.00000
- joint left_foot_ry: limit lower=-0.52360 upper=0.52360 effort=1000.00000 velocity=0.00000 -> lower=-3.14000 upper=3.14000 effort=100.0 velocity=1.00000
- joint left_foot_rz: limit lower=-0.52360 upper=0.52360 effort=0.00000 velocity=0.00000 -> lower=-3.14000 upper=3.14000 effort=0.00000 velocity=1.00000
- joint left_hand_rx: limit lower=-0.52360 upper=0.52360 effort=1000.00000 velocity=0.00000 -> lower=-3.14000 upper=3.14000 effort=100.0 velocity=1.00000
- joint left_hand_ry: limit lower=-0.52360 upper=0.52360 effort=1000.00000 velocity=0.00000 -> lower=-3.14000 upper=3.14000 effort=100.0 velocity=1.00000
- joint left_hand_rz: limit lower=-0.52360 upper=0.52360 effort=1000.00000 velocity=0.00000 -> lower=-3.14000 upper=3.14000 effort=100.0 velocity=1.00000
- joint left_hip_rx: limit lower=-1.57080 upper=0.31067 effort=1000.00000 velocity=0.00000 -> lower=-3.14000 upper=3.14000 effort=100.0 velocity=1.00000
- joint left_hip_ry: limit lower=-0.58818 upper=0.56898 effort=1000.00000 velocity=0.00000 -> lower=-3.14000 upper=3.14000 effort=100.0 velocity=1.00000
- joint left_hip_rz: limit lower=-0.53233 upper=0.67370 effort=1000.00000 velocity=0.00000 -> lower=-3.14000 upper=3.14000 effort=100.0 velocity=1.00000
- joint left_knee_rx: limit lower=-0.02269 upper=2.44172 effort=1000.00000 velocity=0.00000 -> lower=-3.14000 upper=3.14000 effort=100.0 velocity=1.00000
- joint left_knee_ry: limit lower=0.00000 upper=0.00000 effort=1000.00000 velocity=0.00000 -> lower=-3.14000 upper=3.14000 effort=100.0 velocity=1.00000
- joint left_knee_rz: limit lower=0.00000 upper=0.00000 effort=1000.00000 velocity=0.00000 -> lower=-3.14000 upper=3.14000 effort=100.0 velocity=1.00000
- joint left_lowarm_rx: limit lower=-0.52360 upper=0.52360 effort=1000.00000 velocity=0.00000 -> lower=-3.14000 upper=3.14000 effort=100.0 velocity=1.00000
- joint left_lowarm_ry: limit lower=-0.52360 upper=0.52360 effort=1000.00000 velocity=0.00000 -> lower=-3.14000 upper=3.14000 effort=100.0 velocity=1.00000
- joint left_lowarm_rz: limit lower=-0.52360 upper=0.52360 effort=1000.00000 velocity=0.00000 -> lower=-3.14000 upper=3.14000 effort=100.0 velocity=1.00000
- joint left_shoulder_rx: limit lower=-1.03440 upper=0.94713 effort=1000.00000 velocity=0.00000 -> lower=-3.14000 upper=3.14000 effort=100.0 velocity=1.00000
- joint left_shoulder_ry: limit lower=-1.63712 upper=0.50847 effort=1000.00000 velocity=0.00000 -> lower=-3.14000 upper=3.14000 effort=100.0 velocity=1.00000
- joint left_shoulder_rz: limit lower=-1.04720 upper=0.93550 effort=1000.00000 velocity=0.00000 -> lower=-3.14000 upper=3.14000 effort=100.0 velocity=1.00000
- joint neck_rx: limit lower=-0.52360 upper=0.52360 effort=1000.00000 velocity=0.00000 -> lower=-3.14000 upper=3.14000 effort=100.0 velocity=1.00000
- joint neck_ry: limit lower=-0.08727 upper=0.08727 effort=1000.00000 velocity=0.00000 -> lower=-3.14000 upper=3.14000 effort=100.0 velocity=1.00000
- joint neck_rz: limit lower=-0.08727 upper=0.08727 effort=1000.00000 velocity=0.00000 -> lower=-3.14000 upper=3.14000 effort=100.0 velocity=1.00000
- joint right_ankle_rx: limit lower=-0.52360 upper=0.52360 effort=1000.00000 velocity=0.00000 -> lower=-3.14000 upper=3.14000 effort=100.0 velocity=1.00000
- joint right_ankle_ry: limit lower=-0.52360 upper=0.52360 effort=1000.00000 velocity=0.00000 -> lower=-3.14000 upper=3.14000 effort=100.0 velocity=1.00000
- joint right_ankle_rz: limit lower=-0.52360 upper=0.52360 effort=1000.00000 velocity=0.00000 -> lower=-3.14000 upper=3.14000 effort=100.0 velocity=1.00000
- joint right_clavicle_rx: limit lower=-0.51720 upper=0.47357 effort=1000.00000 velocity=0.00000 -> lower=-3.14000 upper=3.14000 effort=100.0 velocity=1.00000
- joint right_clavicle_ry: limit lower=-0.25424 upper=0.81856 effort=1000.00000 velocity=0.00000 -> lower=-3.14000 upper=3.14000 effort=100.0 velocity=1.00000
- joint right_clavicle_rz: limit lower=-0.52360 upper=0.46775 effort=1000.00000 velocity=0.00000 -> lower=-3.14000 upper=3.14000 effort=100.0 velocity=1.00000
- joint right_elbow_rx: limit lower=0.00000 upper=0.00000 effort=1000.00000 velocity=0.00000 -> lower=-3.14000 upper=3.14000 effort=100.0 velocity=1.00000
- joint right_elbow_ry: limit lower=-0.04887 upper=2.57087 effort=1000.00000 velocity=0.00000 -> lower=-3.14000 upper=3.14000 effort=100.0 velocity=1.00000
- joint right_elbow_rz: limit lower=0.00000 upper=0.00000 effort=1000.00000 velocity=0.00000 -> lower=-3.14000 upper=3.14000 effort=100.0 velocity=1.00000
- joint right_foot_rx: limit lower=-0.52360 upper=0.52360 effort=1000.00000 velocity=0.00000 -> lower=-3.14000 upper=3.14000 effort=100.0 velocity=1.00000
- joint right_foot_ry: limit lower=-0.52360 upper=0.52360 effort=1000.00000 velocity=0.00000 -> lower=-3.14000 upper=3.14000 effort=100.0 velocity=1.00000
- joint right_foot_rz: limit lower=-0.52360 upper=0.52360 effort=1000.00000 velocity=0.00000 -> lower=-3.14000 upper=3.14000 effort=100.0 velocity=1.00000
- joint right_hand_rx: limit lower=-0.52360 upper=0.52360 effort=1000.00000 velocity=0.00000 -> lower=-3.14000 upper=3.14000 effort=100.0 velocity=1.00000
- joint right_hand_ry: limit lower=-0.52360 upper=0.52360 effort=1000.00000 velocity=0.00000 -> lower=-3.14000 upper=3.14000 effort=100.0 velocity=1.00000
- joint right_hand_rz: limit lower=-0.52360 upper=0.52360 effort=1000.00000 velocity=0.00000 -> lower=-3.14000 upper=3.14000 effort=100.0 velocity=1.00000
- joint right_hip_rx: limit lower=-1.57080 upper=0.31067 effort=1000.00000 velocity=0.00000 -> lower=-3.14000 upper=3.14000 effort=100.0 velocity=1.00000
- joint right_hip_ry: limit lower=-0.56898 upper=0.58818 effort=1000.00000 velocity=0.00000 -> lower=-3.14000 upper=3.14000 effort=100.0 velocity=1.00000
- joint right_hip_rz: limit lower=-0.67370 upper=0.53233 effort=1000.00000 velocity=0.00000 -> lower=-3.14000 upper=3.14000 effort=100.0 velocity=1.00000
- joint right_knee_rx: limit lower=-0.02269 upper=2.44172 effort=1000.00000 velocity=0.00000 -> lower=-3.14000 upper=3.14000 effort=100.0 velocity=1.00000
- joint right_knee_ry: limit lower=0.00000 upper=0.00000 effort=1000.00000 velocity=0.00000 -> lower=-3.14000 upper=3.14000 effort=100.0 velocity=1.00000
- joint right_knee_rz: limit lower=0.00000 upper=0.00000 effort=1000.00000 velocity=0.00000 -> lower=-3.14000 upper=3.14000 effort=100.0 velocity=1.00000
- joint right_lowarm_rx: limit lower=-0.52360 upper=0.52360 effort=1000.00000 velocity=0.00000 -> lower=-3.14000 upper=3.14000 effort=100.0 velocity=1.00000
- joint right_lowarm_ry: limit lower=-0.52360 upper=0.52360 effort=1000.00000 velocity=0.00000 -> lower=-3.14000 upper=3.14000 effort=100.0 velocity=1.00000
- joint right_lowarm_rz: limit lower=-0.52360 upper=0.52360 effort=1000.00000 velocity=0.00000 -> lower=-3.14000 upper=3.14000 effort=100.0 velocity=1.00000
- joint right_shoulder_rx: limit lower=-1.03440 upper=0.94713 effort=1000.00000 velocity=0.00000 -> lower=-3.14000 upper=3.14000 effort=100.0 velocity=1.00000
- joint right_shoulder_ry: limit lower=-0.50847 upper=1.63712 effort=1000.00000 velocity=0.00000 -> lower=-3.14000 upper=3.14000 effort=100.0 velocity=1.00000
- joint right_shoulder_rz: limit lower=-1.04720 upper=0.93550 effort=1000.00000 velocity=0.00000 -> lower=-3.14000 upper=3.14000 effort=100.0 velocity=1.00000
- joint spine_2_rx: limit lower=-0.52360 upper=0.52360 effort=1000.00000 velocity=0.00000 -> lower=-3.14000 upper=3.14000 effort=100.0 velocity=1.00000
- joint spine_2_ry: limit lower=-0.52360 upper=0.52360 effort=1000.00000 velocity=0.00000 -> lower=-3.14000 upper=3.14000 effort=100.0 velocity=1.00000
- joint spine_2_rz: limit lower=-0.52360 upper=0.52360 effort=1000.00000 velocity=0.00000 -> lower=-3.14000 upper=3.14000 effort=100.0 velocity=1.00000
- joint spine_3_rx: limit lower=-0.52360 upper=0.52360 effort=1000.00000 velocity=0.00000 -> lower=-3.14000 upper=3.14000 effort=100.0 velocity=1.00000
- joint spine_3_ry: limit lower=-0.52360 upper=0.52360 effort=1000.00000 velocity=0.00000 -> lower=-3.14000 upper=3.14000 effort=100.0 velocity=1.00000
- joint spine_3_rz: limit lower=-0.52360 upper=0.52360 effort=1000.00000 velocity=0.00000 -> lower=-3.14000 upper=3.14000 effort=100.0 velocity=1.00000
- joint spine_4_rx: limit lower=-0.52360 upper=0.52360 effort=1000.00000 velocity=0.00000 -> lower=-3.14000 upper=3.14000 effort=100.0 velocity=1.00000
- joint spine_4_ry: limit lower=-0.52360 upper=0.52360 effort=1000.00000 velocity=0.00000 -> lower=-3.14000 upper=3.14000 effort=100.0 velocity=1.00000
- joint spine_4_rz: limit lower=-0.52360 upper=0.52360 effort=1000.00000 velocity=0.00000 -> lower=-3.14000 upper=3.14000 effort=100.0 velocity=1.00000
